Commit message: finish lab5

File: misc/Lab5/Bipe3D/yanshee/robots/yanshee.urdf (robot description, URDF)
Before this commit: robot yanshee, 19 links, 18 joints
Joints:
- joint left_leg1_joint: type revolute -> fixed
- joint left_leg4_joint: type fixed -> revolute
- joint right_leg1_joint: type revolute -> fixed
- joint right_leg4_joint: type fixed -> revolute
